Commit message: ROboot up to the diffdrive and roscontrol stage

File: description/gazebo_control.xacro (robot description, xacro)
@@ -6,5 +6,5 @@
             <left_joint>left_wheel_joint</left_joint>
             <right_joint>right_wheel_joint</right_joint>
-            <wheel_separation>0.35</wheel_separation>
+            <wheel_separation>0.6</wheel_separation>
             <wheel_radius>0.05</wheel_radius>
             <!-- Input -->

File: description/lidar.xacro (robot description, xacro)
@@ -4,5 +4,5 @@
         <parent link="chassis"/>
         <child link="laser_frame"/>
-        <origin xyz="0.1 0 0.175" rpy="0 0 0"/>
+        <origin xyz="0.1 0 0.3" rpy="0 0 0"/>
     </joint>
     <link name="laser_frame">
@@ -25,6 +25,6 @@
         <sensor name="laser" type="gpu_lidar">
             <pose> 0 0 0 0 0 0 </pose>
-            <visualize>false</visualize>
             <update_rate>10</update_rate>
+            <topic>scan</topic>
             <lidar>
                 <scan>
@@ -40,6 +40,6 @@
                 </range>
             </lidar>
-            <topic>scan</topic>
-            <gz_frame_id>laser_frame</gz_frame_id>
+            <always_on>1</always_on>
+            <visualize>1</visualize>
         </sensor>
     </gazebo>

File: description/robot.urdf.xacro (robot description, xacro)
@@ -1,6 +1,14 @@
 <?xml version="1.0"?>
 <robot xmlns:xacro="http://www.ros.org/wiki/xacro"  name="robot">
+    <xacro:arg name="use_ros2_control" default="true"/>
     <xacro:include filename="robot_core.xacro" />
-    <xacro:include filename="gazebo_control.xacro"/>
+          <!-- Switch between ros2_control and Gazebo integrated diff-drive control -->
+    <xacro:if value="$(arg use_ros2_control)">
+        <xacro:include filename="ros2_control.xacro" />
+    </xacro:if>
+    <xacro:unless value="$(arg use_ros2_control)">
+        <xacro:include filename="gazebo_control.xacro" />
+    </xacro:unless>
+    <xacro:include filename="ros2_control.xacro"/>
     <xacro:include filename="lidar.xacro" />
 </robot>

File: description/robot_core.xacro (robot description, xacro)
@@ -29,5 +29,5 @@
             <origin xyz="0.15 0 0.075" rpy="0 0 0"/>
             <geometry>
-                <box size="0.3 0.3 0.15"/>
+                <cylinder length="0.3" radius="0.5"/>
             </geometry>
             <material name="white"/>
@@ -36,10 +36,79 @@
             <origin xyz="0.15 0 0.075" rpy="0 0 0"/>
             <geometry>
-                <box size="0.3 0.3 0.15"/>
+                <cylinder length="0.3" radius="0.5"/>
             </geometry>
         </collision>
-        <xacro:inertial_box mass="0.5" x="0.3" y="0.3" z="0.15">
+        <xacro:inertial_cylinder mass="0.5" length="0.3" radius="0.5">
             <origin xyz="0.15 0 0.075" rpy="0 0 0"/>
-        </xacro:inertial_box>
+        </xacro:inertial_cylinder>
+    </link>
+    <joint name="badboy0" type="fixed">
+        <parent link="chassis"/>
+        <child link="badboy_link0"/>
+        <origin xyz="-0.2 0 0.3"/>
+    </joint>
+    <link name="badboy_link0">
+        <visual>
+            <origin xyz="-0.2 0 0.3" rpy="0 0 0"/>
+            <geometry>
+                <cylinder length="1" radius="0.005"/>
+            </geometry>
+            <material name="white"/>
+        </visual>
+        <collision>
+            <origin xyz="-0.2 0 0.3" rpy="0 0 0"/>
+            <geometry>
+                <cylinder length="1" radius="0.005"/>
+            </geometry>
+        </collision>
+        <xacro:inertial_cylinder mass="0.1" length="1" radius="0.005">
+            <origin xyz="-0.2 0 0.3" rpy="0 0 0"/>
+        </xacro:inertial_cylinder>
+    </link>
+    <joint name="badboy1" type="fixed">
+        <parent link="chassis"/>
+        <child link="badboy_link1"/>
+        <origin xyz="0.2 0.2 0.3"/>
+    </joint>
+    <link name="badboy_link1">
+        <visual>
+            <origin xyz="0.2 0.2 0.3" rpy="0 0 0"/>
+            <geometry>
+                <cylinder length="1" radius="0.005"/>
+            </geometry>
+            <material name="white"/>
+        </visual>
+        <collision>
+            <origin xyz="0.2 0.2 0.3" rpy="0 0 0"/>
+            <geometry>
+                <cylinder length="1" radius="0.005"/>
+            </geometry>
+        </collision>
+        <xacro:inertial_cylinder mass="0.1" length="1" radius="0.005">
+            <origin xyz="0.2 0.2 0.3" rpy="0 0 0"/>
+        </xacro:inertial_cylinder>
+    </link>
+    <joint name="badboy2" type="fixed">
+        <parent link="chassis"/>
+        <child link="badboy_link2"/>
+        <origin xyz="0.2 -0.2 0.3"/>
+    </joint>
+    <link name="badboy_link2">
+        <visual>
+            <origin xyz="0.2 -0.2 0.3" rpy="0 0 0"/>
+            <geometry>
+                <cylinder length="1" radius="0.005"/>
+            </geometry>
+            <material name="white"/>
+        </visual>
+        <collision>
+            <origin xyz="0.2 -0.2 0.3" rpy="0 0 0"/>
+            <geometry>
+                <cylinder length="1" radius="0.005"/>
+            </geometry>
+        </collision>
+        <xacro:inertial_cylinder mass="0.1" length="1" radius="0.005">
+            <origin xyz="0.2 -0.2 0.3" rpy="0 0 0"/>
+        </xacro:inertial_cylinder>
     </link>
     <!-- LEFT WHEEL -->
@@ -47,5 +116,5 @@
         <parent link="base_link"/>
         <child link="left_wheel"/>
-        <origin xyz="0 0.15 0" rpy="-${pi/2} 0 0"/>
+        <origin xyz="0 0.3 0" rpy="-${pi/2} 0 0"/>
         <axis xyz="0 0 1"/>
         <limit effort="0.05" velocity="10.0"/>
@@ -71,5 +140,5 @@
         <parent link="base_link"/>
         <child link="right_wheel"/>
-        <origin xyz="0 -0.15 0" rpy="${pi/2} 0 0"/>
+        <origin xyz="0 -0.3 0" rpy="${pi/2} 0 0"/>
         <axis xyz="0 0 -1"/>
         <limit effort="0.05" velocity="10.0"/>

Commit message: pi

File: description/gazebo_control.xacro (robot description, xacro)
@@ -7,5 +7,5 @@
             <right_joint>right_wheel_joint</right_joint>
             <wheel_separation>0.6</wheel_separation>
-            <wheel_radius>0.05</wheel_radius>
+            <wheel_radius>0.075</wheel_radius>
             <!-- Input -->
             <topic>cmd_vel</topic>

File: description/robot_core.xacro (robot description, xacro)
@@ -19,5 +19,5 @@
     <link name="base_link">
     </link>
-        <!-- BASE_FOOTPRINT -->
+    <!-- BASE_FOOTPRINT -->
     <joint name="base_footprint_joint" type="fixed">
         <parent link="base_link"/>
@@ -37,5 +37,5 @@
             <origin xyz="0.15 0 0.075" rpy="0 0 0"/>
             <geometry>
-                <cylinder length="0.3" radius="0.5"/>
+                <cylinder length="0.3" radius="0.3"/>
             </geometry>
             <material name="white"/>
@@ -44,8 +44,8 @@
             <origin xyz="0.15 0 0.075" rpy="0 0 0"/>
             <geometry>
-                <cylinder length="0.3" radius="0.5"/>
+                <cylinder length="0.3" radius="0.3"/>
             </geometry>
         </collision>
-        <xacro:inertial_cylinder mass="0.5" length="0.3" radius="0.5">
+        <xacro:inertial_cylinder mass="0.5" length="0.3" radius="0.3">
             <origin xyz="0.15 0 0.075" rpy="0 0 0"/>
         </xacro:inertial_cylinder>
@@ -131,5 +131,5 @@
         <visual>
             <geometry>
-                <cylinder length="0.04" radius="0.05" />
+                <cylinder length="0.04" radius="0.075" />
             </geometry>
             <material name="blue"/>
@@ -140,5 +140,5 @@
             </geometry>
         </collision>
-        <xacro:inertial_cylinder mass="0.1" length="0.04" radius="0.05">
+        <xacro:inertial_cylinder mass="0.1" length="0.04" radius="0.075">
             <origin xyz="0 0 0" rpy="0 0 0"/>
         </xacro:inertial_cylinder>
@@ -155,5 +155,5 @@
         <visual>
             <geometry>
-                <cylinder length="0.04" radius="0.05" />
+                <cylinder length="0.04" radius="0.075" />
             </geometry>
             <material name="blue"/>
@@ -164,5 +164,5 @@
             </geometry>
         </collision>
-        <xacro:inertial_cylinder mass="0.1" length="0.04" radius="0.05">
+        <xacro:inertial_cylinder mass="0.1" length="0.04" radius="0.075">
             <origin xyz="0 0 0" rpy="0 0 0"/>
         </xacro:inertial_cylinder>
