Commit message: hello welcome to pi

File: description/robot_core.xacro (robot description, xacro)
@@ -18,4 +18,12 @@
     </material>
     <link name="base_link">
+    </link>
+        <!-- BASE_FOOTPRINT -->
+    <joint name="base_footprint_joint" type="fixed">
+        <parent link="base_link"/>
+        <child link="base_footprint"/>
+        <origin xyz="0 0 0" rpy="0 0 0"/>
+    </joint>
+    <link name="base_footprint">
     </link>
     <!-- CHASSIS -->

Commit message: pi

File: description/robot_core.xacro (robot description, xacro)
@@ -1,13 +1,24 @@
 <?xml version="1.0"?>
-<robot xmlns:xacro="http://www.ros.org/wiki/xacro">
-    <xacro:include filename="inertial_macros.xacro" />
+<robot xmlns:xacro="http://www.ros.org/wiki/xacro" >
+    <xacro:include filename="inertial_macros.xacro"/>
+    <xacro:property name="chassis_length" value="0.6"/>
+    <xacro:property name="chassis_width" value="0.6"/>
+    <xacro:property name="chassis_height" value="0.138"/>
+    <xacro:property name="chassis_mass" value="1.0"/>
+    <xacro:property name="wheel_radius" value="0.075"/>
+    <xacro:property name="wheel_thickness" value="0.026"/>
+    <xacro:property name="wheel_mass" value="0.05"/>
+    <xacro:property name="wheel_offset_x" value="0.226"/>
+    <xacro:property name="wheel_offset_y" value="0.1485"/>
+    <xacro:property name="wheel_offset_z" value="0.01"/>
+    <xacro:property name="caster_wheel_radius" value="0.01"/>
+    <xacro:property name="caster_wheel_mass" value="0.01"/>
+    <xacro:property name="caster_wheel_offset_x" value="0.075"/>
+    <xacro:property name="caster_wheel_offset_z" value="${wheel_offset_z - wheel_radius + caster_wheel_radius}"/>
     <material name="white">
-        <color rgba="1 1 1 1"/>
+        <color rgba="1 1 1 1" />
     </material>
     <material name="orange">
         <color rgba="1 0.3 0.1 1"/>
-    </material>
-    <material name="red">
-        <color rgba="1 0 0 1"/>
     </material>
     <material name="blue">
@@ -17,7 +28,11 @@
         <color rgba="0 0 0 1"/>
     </material>
+    <material name="red">
+        <color rgba="1 0 0 1"/>
+    </material>
+    <!-- BASE LINK -->
     <link name="base_link">
     </link>
-    <!-- BASE_FOOTPRINT -->
+    <!-- BASE_FOOTPRINT LINK -->
     <joint name="base_footprint_joint" type="fixed">
         <parent link="base_link"/>
@@ -27,109 +42,42 @@
     <link name="base_footprint">
     </link>
-    <!-- CHASSIS -->
+    <!-- CHASSIS LINK -->
     <joint name="chassis_joint" type="fixed">
         <parent link="base_link"/>
         <child link="chassis"/>
-        <origin xyz="-0.1 0 0"/>
+        <origin xyz="${-wheel_offset_x} 0 ${-wheel_offset_z}"/>
     </joint>
     <link name="chassis">
         <visual>
-            <origin xyz="0.15 0 0.075" rpy="0 0 0"/>
+            <origin xyz="${chassis_length/2} 0 ${chassis_height/2}"/>
             <geometry>
-                <cylinder length="0.3" radius="0.3"/>
+                <box size="${chassis_length} ${chassis_width} ${chassis_height}"/>
             </geometry>
-            <material name="white"/>
+            <material name="orange"/>
         </visual>
         <collision>
-            <origin xyz="0.15 0 0.075" rpy="0 0 0"/>
+            <origin xyz="${chassis_length/2} 0 ${chassis_height/2}"/>
             <geometry>
-                <cylinder length="0.3" radius="0.3"/>
+                <box size="${chassis_length} ${chassis_width} ${chassis_height}"/>
             </geometry>
         </collision>
-        <xacro:inertial_cylinder mass="0.5" length="0.3" radius="0.3">
-            <origin xyz="0.15 0 0.075" rpy="0 0 0"/>
-        </xacro:inertial_cylinder>
+        <xacro:inertial_box mass="0.5" x="${chassis_length}" y="${chassis_width}" z="${chassis_height}">
+            <origin xyz="${chassis_length/2} 0 ${chassis_height/2}" rpy="0 0 0"/>
+        </xacro:inertial_box>
     </link>
-    <joint name="badboy0" type="fixed">
-        <parent link="chassis"/>
-        <child link="badboy_link0"/>
-        <origin xyz="-0.2 0 0.3"/>
-    </joint>
-    <link name="badboy_link0">
-        <visual>
-            <origin xyz="-0.2 0 0.3" rpy="0 0 0"/>
-            <geometry>
-                <cylinder length="1" radius="0.005"/>
-            </geometry>
-            <material name="white"/>
-        </visual>
-        <collision>
-            <origin xyz="-0.2 0 0.3" rpy="0 0 0"/>
-            <geometry>
-                <cylinder length="1" radius="0.005"/>
-            </geometry>
-        </collision>
-        <xacro:inertial_cylinder mass="0.1" length="1" radius="0.005">
-            <origin xyz="-0.2 0 0.3" rpy="0 0 0"/>
-        </xacro:inertial_cylinder>
-    </link>
-    <joint name="badboy1" type="fixed">
-        <parent link="chassis"/>
-        <child link="badboy_link1"/>
-        <origin xyz="0.2 0.2 0.3"/>
-    </joint>
-    <link name="badboy_link1">
-        <visual>
-            <origin xyz="0.2 0.2 0.3" rpy="0 0 0"/>
-            <geometry>
-                <cylinder length="1" radius="0.005"/>
-            </geometry>
-            <material name="white"/>
-        </visual>
-        <collision>
-            <origin xyz="0.2 0.2 0.3" rpy="0 0 0"/>
-            <geometry>
-                <cylinder length="1" radius="0.005"/>
-            </geometry>
-        </collision>
-        <xacro:inertial_cylinder mass="0.1" length="1" radius="0.005">
-            <origin xyz="0.2 0.2 0.3" rpy="0 0 0"/>
-        </xacro:inertial_cylinder>
-    </link>
-    <joint name="badboy2" type="fixed">
-        <parent link="chassis"/>
-        <child link="badboy_link2"/>
-        <origin xyz="0.2 -0.2 0.3"/>
-    </joint>
-    <link name="badboy_link2">
-        <visual>
-            <origin xyz="0.2 -0.2 0.3" rpy="0 0 0"/>
-            <geometry>
-                <cylinder length="1" radius="0.005"/>
-            </geometry>
-            <material name="white"/>
-        </visual>
-        <collision>
-            <origin xyz="0.2 -0.2 0.3" rpy="0 0 0"/>
-            <geometry>
-                <cylinder length="1" radius="0.005"/>
-            </geometry>
-        </collision>
-        <xacro:inertial_cylinder mass="0.1" length="1" radius="0.005">
-            <origin xyz="0.2 -0.2 0.3" rpy="0 0 0"/>
-        </xacro:inertial_cylinder>
-    </link>
-    <!-- LEFT WHEEL -->
+    <gazebo reference="chassis">
+        <material>Gazebo/Orange</material>
+    </gazebo>
+    <!-- LEFT WHEEL LINK -->
     <joint name="left_wheel_joint" type="continuous">
         <parent link="base_link"/>
         <child link="left_wheel"/>
-        <origin xyz="0 0.3 0" rpy="-${pi/2} 0 0"/>
+        <origin xyz="0 ${wheel_offset_y} 0" rpy="-${pi/2} 0 0" />
         <axis xyz="0 0 1"/>
-        <limit effort="0.05" velocity="10.0"/>
     </joint>
     <link name="left_wheel">
         <visual>
             <geometry>
-                <cylinder length="0.04" radius="0.075" />
+                <cylinder radius="${wheel_radius}" length="${wheel_thickness}"/>
             </geometry>
             <material name="blue"/>
@@ -137,23 +85,25 @@
         <collision>
             <geometry>
-                <sphere radius="0.05" />
+                <sphere radius="${wheel_radius}"/>
             </geometry>
         </collision>
-        <xacro:inertial_cylinder mass="0.1" length="0.04" radius="0.075">
+        <xacro:inertial_cylinder mass="${wheel_mass}" length="${wheel_thickness}" radius="${wheel_radius}">
             <origin xyz="0 0 0" rpy="0 0 0"/>
         </xacro:inertial_cylinder>
     </link>
-    <!-- RIGHT WHEEL -->
+    <gazebo reference="left_wheel">
+        <material>Gazebo/Blue</material>
+    </gazebo>
+    <!-- RIGHT WHEEL LINK -->
     <joint name="right_wheel_joint" type="continuous">
         <parent link="base_link"/>
         <child link="right_wheel"/>
-        <origin xyz="0 -0.3 0" rpy="${pi/2} 0 0"/>
+        <origin xyz="0 ${-wheel_offset_y} 0" rpy="${pi/2} 0 0" />
         <axis xyz="0 0 -1"/>
-        <limit effort="0.05" velocity="10.0"/>
     </joint>
     <link name="right_wheel">
         <visual>
             <geometry>
-                <cylinder length="0.04" radius="0.075" />
+                <cylinder radius="${wheel_radius}" length="${wheel_thickness}"/>
             </geometry>
             <material name="blue"/>
@@ -161,36 +111,40 @@
         <collision>
             <geometry>
-                <sphere radius="0.05" />
+                <sphere radius="${wheel_radius}"/>
             </geometry>
         </collision>
-        <xacro:inertial_cylinder mass="0.1" length="0.04" radius="0.075">
+        <xacro:inertial_cylinder mass="${wheel_mass}" length="${wheel_thickness}" radius="${wheel_radius}">
             <origin xyz="0 0 0" rpy="0 0 0"/>
         </xacro:inertial_cylinder>
     </link>
-    <!-- CASTER WHEEL -->
+    <gazebo reference="right_wheel">
+        <material>Gazebo/Blue</material>
+    </gazebo>
+    <!-- CASTER WHEEL LINK -->
     <joint name="caster_wheel_joint" type="fixed">
         <parent link="chassis"/>
         <child link="caster_wheel"/>
-        <origin xyz="0.24 0 0" rpy="0 0 0"/>
+        <origin xyz="${caster_wheel_offset_x} 0 ${caster_wheel_offset_z}"/>
     </joint>
     <link name="caster_wheel">
         <visual>
             <geometry>
-                <sphere radius="0.05" />
+                <sphere radius="${caster_wheel_radius}"/>
             </geometry>
-            <material name="black"/>
+            <material name="white"/>
         </visual>
         <collision>
             <geometry>
-                <sphere radius="0.05" />
+                <sphere radius="${caster_wheel_radius}"/>
             </geometry>
         </collision>
-        <xacro:inertial_sphere mass="0.1" radius="0.05">
+        <xacro:inertial_sphere mass="${caster_wheel_mass}" radius="${caster_wheel_radius}">
             <origin xyz="0 0 0" rpy="0 0 0"/>
         </xacro:inertial_sphere>
     </link>
     <gazebo reference="caster_wheel">
-        <mu1 value="0.0"/>
-        <mu2 value="0.0"/>
+        <material>Gazebo/White</material>
+        <mu1 value="0.001"/>
+        <mu2 value="0.001"/>
     </gazebo>
 </robot>

File: description/ros2_control.xacro (robot description, xacro)
@@ -28,4 +28,5 @@
                         <!-- Make sure to put your package name in there!! -->
             <parameters>$(find my_bot)/config/my_controllers.yaml</parameters>
+        </plugin>
     </gazebo>
         </xacro:if>
