Commit message: newest

File: description/robot.urdf.xacro (robot description, xacro)
@@ -10,5 +10,7 @@
         <xacro:include filename="gazebo_control.xacro" />
     </xacro:unless>
-    <xacro:include filename="ros2_control.xacro"/>
+    <!-- <xacro:include filename="ros2_control.xacro"/> -->
     <xacro:include filename="lidar.xacro" />
+    <xacro:include filename="tripod.xacro"/>
+    <xacro:include filename="camera.xacro"/>
 </robot>

File: description/robot_core.xacro (robot description, xacro)
@@ -4,12 +4,12 @@
     <xacro:property name="chassis_length" value="0.6"/>
     <xacro:property name="chassis_width" value="0.6"/>
-    <xacro:property name="chassis_height" value="0.138"/>
+    <xacro:property name="chassis_height" value="0.005"/>
     <xacro:property name="chassis_mass" value="1.0"/>
     <xacro:property name="wheel_radius" value="0.075"/>
     <xacro:property name="wheel_thickness" value="0.026"/>
     <xacro:property name="wheel_mass" value="0.05"/>
-    <xacro:property name="wheel_offset_x" value="0.226"/>
-    <xacro:property name="wheel_offset_y" value="0.1485"/>
-    <xacro:property name="wheel_offset_z" value="0.01"/>
+    <xacro:property name="wheel_offset_x" value="0.3"/>
+    <xacro:property name="wheel_offset_y" value="0.3"/>
+    <xacro:property name="wheel_offset_z" value="0.05"/>
     <xacro:property name="caster_wheel_radius" value="0.01"/>
     <xacro:property name="caster_wheel_mass" value="0.01"/>
